File: pcb/TofStand.sch (KiCad schematic (older format))
At the start: 83 parts, among them SW2 SWITCH_H, U1 L6470

Commit message: Proceeding
Connections:
- wire segments 293 -> 294
- no-connect marks 40 -> 39
Other:
- note added: "0 at this PCB, 1 at old PCB"
Changed lines of the file:
@@
 NoConn ~ 6750 3650
 NoConn ~ 6750 3750
-NoConn ~ 6750 3850
 NoConn ~ 6750 3950
 NoConn ~ 6750 4350
@@
 	1    0    0    -1
 $EndComp
+$Comp
+L power:GND #PWR?
+U 1 1 5D7254FA
+P 6850 3850
+F 0 "#PWR?" H 6940 3830 30  0001 C CNN
+F 1 "GND" H 6850 3770 30  0001 C CNN
+F 2 "" H 6850 3850 60  0000 C CNN
+F 3 "" H 6850 3850 60  0000 C CNN
+	1    6850 3850
+	0    1    1    0
+$EndComp
+Wire Wire Line
+	6850 3850 6750 3850
+Text Notes 6900 3850 0    50   ~ 0
+0 at this PCB, 1 at old PCB
 $EndSCHEMATC

Commit message: PCB sent to factory
Parts:
- removed C48: 1000u, Capacitors:CAP_10xxR, symbol Tittar_kl:CP
- removed HOLE3, HOLE9: HOLE_METALLED, PCB:Hole3_5_out6mm, symbol pcb_details:HOLE_METALLED
- DA1: footprint SO_DIL_TSSOP:SO8 -> SO_DIL_TSSOP:SO8_150MIL
- XL1: renamed from XL?; footprint Connectors:PLS-6-NoHole -> Connectors:PLS-6
- XL2: renamed from XL?; footprint Connectors:uUSB_614105150721 -> Connectors:USBmicro_MOLEX_1050170001
- gave numbers to parts that had none: 18
Connections:
- wire segments 294 -> 288

Commit message: + PCB v2 + Release firmwares
Parts:
- removed D1, D2: 1N4148, Diodes:SOD80C, symbol Tittar_kl:DIODE
- removed DD1: STM32F405RX-64, LQFP_TQFP:LQFP64, symbol st_kl:STM32F405Rx-64
- removed VCap1, VCap2: 2.2u, Capacitors:CAP_0603, symbol Tittar_kl:C
- added DD1: STM32F103RC-64, LQFP_TQFP:LQFP64, symbol st_kl:STM32F103RC-64
- added R5: 1k5, Resistors:RES_0603, symbol Tittar_kl:R
Connections:
- net labels added: USB_PULLUP
- wire segments 288 -> 287
- no-connect marks 39 -> 37
Other:
- note removed: "0 at this PCB, 1 at old PCB"
- moved on the sheet: C10, C11, C12, C13, C14, C15, C7, C8, C9, D4, R3, R4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

Commit message: + V2.0 Sch done
Parts:
- removed D4: LED, LEDs:LED_0603, symbol Tittar_kl:LED
- removed DA1: LP2951, SO_DIL_TSSOP:SO8_150MIL, symbol Power_kl:LP2951
- removed DD1: STM32F103RC-64, LQFP_TQFP:LQFP64, symbol st_kl:STM32F103RC-64
- removed HOLE10, HOLE6, HOLE8: HOLE_METALLED, PCB:Hole3_5_out6mm, symbol pcb_details:HOLE_METALLED
- removed R51: 20k, Resistors:RES_0603, symbol Tittar_kl:R
- removed R52: 12k, Resistors:RES_0603, symbol Tittar_kl:R
- removed R53: 1k, Resistors:RES_0603, symbol Tittar_kl:R
- removed SW2: SWITCH_H, BtnsSwitches:SW_SS9, symbol Switches:SWITCH_H
- removed XL1: CONN_6, Connectors:PLS-6, symbol Connectors_kl:CONN_6
- removed XL4: CONN_3, Connectors:W03_Pitch_2d54, symbol Connectors_kl:CONN_3
- removed XL8: BARREL_SOCKET, Connectors:Barrel, symbol Connectors_kl:BARREL_SOCKET
- added C16, C24, C28, C29, C30, C31, C32, C33, C34, C5: 0.1u, Capacitors:CAP_0603_Silks, symbol Tittar_kl:C
- added C17, C22, C35, C36: 0.1u, Capacitors:CAP_0402, symbol Tittar_kl:C
- added C20, C21, C38, C39: 10u, Capacitors:CAP_0603, symbol Tittar_kl:C
- added C23, C25, C26, C27, C37, C42, C58: 0.1u, Capacitors:CAP_0603, symbol Tittar_kl:C
- added C4: 18pF, Capacitors:CAP_0603_Silks, symbol Tittar_kl:C
- added C40, C43: 1u, Capacitors:CAP_0603, symbol Tittar_kl:C
- added C41: 10n, Capacitors:CAP_0603, symbol Tittar_kl:C
- added C56: 1000u, Capacitors:CAP_10xxR, symbol Tittar_kl:CP
- added D1, D11, D12, D14, D15, D16, D17, D2, D3, D5, D6, D7: PESD3V3, Diodes:SOD323, symbol Tittar_kl:ZenerBidir
- added D10, D13, D9: LED, LEDs:LED_Through-Hole-5mm, symbol Tittar_kl:LED
- added D20, D21, D8: LED, LEDs:LED_0603, symbol Tittar_kl:LED
- added D4: PMEG2020, Diodes:SOD323, symbol Tittar_kl:D_Shottky
- added DA1: SY8120, SOT:SOT23-6, symbol Power_kl:SY8120
- added DA2, DA3, DA4, DA5, DA6, DA7, DA8, DA9: Optocoupler_6N137, symbol Interface_kl:Optocoupler_6N137
- added DD1: STM32F205Rx-64, symbol st_kl:STM32F205Rx-64
- added DD2, DD3: ICN2595, SO_DIL_TSSOP:TSSOP24_150_0635, symbol LED_Driver:ICN2595
- added DD4: 74LVC2G17, symbol standard_logic:74LVC2G17
- added DD5: TUSB211, QFN_DFN:X2QFN_12, symbol Interface_kl:TUSB211
- added HOLE1, HOLE2: HOLE_METALLED, PCB:Hole3_5_out6mm, symbol pcb_details:HOLE_METALLED
- added L1, L6, L9: BLM21PG221SN1D, Inductors:IND_0603, symbol Tittar_kl:L
- added L2: BLM15AG102, Inductors:IND_0402, symbol Tittar_kl:L
- added L3, L7, L8: 90R, Inductors:DLW21SN, symbol Tittar_kl:CHOKE_COIL
- added L4: 2R2, Inductors:IND_1515, symbol Tittar_kl:L
- added L5: Choke, Inductors:IND_0402, symbol Tittar_kl:L
- added Q1, Q2, Q3, Q5: 2N7002, symbol Transistors_kl:N_3PIN
- added Q4: IRF9321, SO_DIL_TSSOP:SO8HEATSINK, symbol Transistors_kl:P_8PIN_W_PAD
- added R10: 22k, Resistors:RES_0402_sm, symbol Tittar_kl:R
- added R11, R16, R17, R27, R28, R29, R45, R7: 100k, Resistors:RES_0603, symbol Tittar_kl:R
- added R12, R13, R14, R15, R18, R19, R20, R21, R22, R23, R24, R25, R30, R31, R32, R33, R34, R40, R41, R6, R8: 1k, Resistors:RES_0603, symbol Tittar_kl:R
- added R26: 10k, Resistors:RES_0603, symbol Tittar_kl:R
- added R35, R36: 1k, Resistors:RES_0402_sm, symbol Tittar_kl:R
- added R37: 3k9, Resistors:RES_0603, symbol Tittar_kl:R
- added R9: 100k, Resistors:RES_0402_sm, symbol Tittar_kl:R
- added SW1, SW2, SW3, SW4: SWT-9, BtnsSwitches:BTN_SWT9, symbol Switches:BUTTON
- added U2, U3: USBLC6, SOT:SOT23-6, symbol ESDProtection:USBLC6
- added VCap1, VCap2: 2.2u, Capacitors:CAP_0603, symbol Tittar_kl:C
- added VD1: 7SEGx4_CA, Display:7Segx4, symbol display_kl:7SEGx4_CA
- added XL1, XL13: CONN_2, symbol Connectors_kl:CONN_2
- added XL10: RASPBERRY_3B, Installation:RaspberryPi3, symbol Connectors_kl:RASPBERRY_3B
- added XL12: USB_MICRO, Connectors:USBmicro_MOLEX_1050170001, symbol Connectors_kl:USB_MICRO_2H
- added XL2: CONN_6, Connectors:PLS-6_LOCK, symbol Connectors_kl:CONN_6
- added XL3: CONN_5, Connectors:PLS-5, symbol Connectors_kl:CONN_5
- added XL5, XL6: CONN_3, Connectors:W03_Pitch_2d54, symbol Connectors_kl:CONN_3
- added XL8: CONN_2, Connectors:WB-02(MW-2M), symbol Connectors_kl:CONN_2
- added XL9: USB_C, symbol Connectors_kl:USB_C
- C1: value 10n -> 18pF; footprint Capacitors:CAP_0603 -> Capacitors:CAP_0603_Silks; Price 0.5 -> (none); SolderPoints 2 -> (none)
- C10: value 18pF -> 10nF; footprint Capacitors:CAP_0603 -> Capacitors:CAP_0603_Silks
- C11, C9: value 0.1u -> 10nF; footprint Capacitors:CAP_0603 -> Capacitors:CAP_0603_Silks
- C12, C8: footprint Capacitors:CAP_0603 -> Capacitors:CAP_0603_Silks
- C13: value 18pF -> 10u; Price (none) -> 0.5; SolderPoints (none) -> 2
- C14: value 0.1u -> 1u; footprint Capacitors:CAP_0603 -> Capacitors:CAP_0402; Price (none) -> 0.5; SolderPoints (none) -> 2
- C15: value 0.1u -> 1u; footprint Capacitors:CAP_0603 -> Capacitors:CAP_0603_Silks
- C18: value 1000pF -> 0.1u; footprint Capacitors:CAP_0603 -> Capacitors:CAP_0402; Price (none) -> 0.5; SolderPoints (none) -> 2
- C19: value 1u -> 27pF; footprint Capacitors:CAP_0603 -> Capacitors:CAP_0402; Price (none) -> 0.5; SolderPoints (none) -> 2
- C2: value 2u2 -> 10u; footprint Capacitors:CAP_0603 -> Capacitors:CAP_0805; Price 0.5 -> (none); SolderPoints 2 -> (none)
- C7: value 10u -> 0.1u; footprint Capacitors:CAP_0805 -> Capacitors:CAP_0603_Silks
- R1: value 1M -> 1k; Comment (none) -> 1% resistor
- R2: value 2R0 -> 1k; Comment (none) -> 1% resistor
- R3: value 10k -> 1k; Comment (none) -> 1% resistor; Price (none) -> 0.5; SolderPoints (none) -> 2
- R46: value 1k -> 10k; Comment (none) -> 1% resistor; Price (none) -> 0.5; SolderPoints (none) -> 2
- R5: value 1k5 -> 56k; footprint Resistors:RES_0603 -> Resistors:RES_0402_sm
- XTAL1: footprint Quartz:0503x4-4 -> Quartz:03225C4
- renumbered C16 to C3, C22 to C44, C24 to C45, C26 to C46, C27 to C47, C30 to C48, C32 to C49, C33 to C50, C36 to C51, C37 to C52, C40 to C53, C42 to C54, C44 to C55, C46 to C57, C17 to C6, D20 to D19, D23 to D22, D25 to D23, HOLE1 to HOLE3, HOLE2 to HOLE4, HOLE4 to HOLE5, HOLE5 to HOLE6, R56 to R38, R58 to R39, R60 to R42, R62 to R43, R64 to R44, R68 to R47, R69 to R48, U2 to U1, U1 to U4, XL17 to XL11, XL3 to XL4, XL2 to XL7
Connections:
- net +12v: now also C56.1, C58.1, XL13.2 (PM); no longer C3.1, C6.1
- net +3v3: now also R46.1, C40.2, C41.2, C43.2, D1.C, D12.C, D2.C, D3.C, DD4.5 (VCC), DD5.12 (Vcc), L2.2, L5.1, R12.2, R19.2, XL5.3, XL6.3; no longer C11.1, C12.1, C14.1, C15.1, C18.1, C19.1, C7.1, C8.1, C9.1, R3.1
- net 5V_USB: now also D4.A, R15.2; no longer R2.1
- net ENDSTOP_BOT: now also C10.1, R2.1, D6.C, DD1.14 ((ADC123-0)/TX4/T5C1/WKUP/PA0)
- net ENDSTOP_TOP: now also C9.1, R1.1, D5.C, DD1.15 ((ADC123-1)/RX4/T5C2/T2C2/PA1); no longer XL4.2 (PM)
- net GND: now also C1.2, XL4.2 (PM), C16.2, C17.2, C20.2, C21.2, C22.2, C23.2, C24.2, C25.2, C26.2, C27.2, C31.2, C32.2, C35.1, C36.1, C37.1, C38.1, C39.1, C4.2, C40.1, C41.1, C42.1, C43.1, C5.2, D1.A, D11.A, D12.A, D14.A, D15.A, D16.A, D17.A, D2.A, D20.C, D21.C, D3.A, D5.A, D6.A, D7.A, D8.C, DA1.2 (GND), DA2.5 (GND), DA3.3 (C), DA4.3 (C), DA5.3 (C), DA6.5 (GND), DA7.5 (GND), DA8.3 (C), DA9.3 (C), DD1.12 (VSSA), DD1.18 (VSS4), DD1.60 (BOOT0), DD1.63 (VSS3), DD2.1 (GND), DD3.1 (GND), DD4.2 (GND), DD5.10 (GND), L1.2, L6.2, L9.2, Q1.2 (S), Q2.2 (S), Q3.2 (S), Q4.PAD, Q5.2 (S), R10.2, R11.2, R16.2, R17.2, R26.2, R27.2, R28.2, R29.2, R35.2, R36.2, R37.2, R45.2, R7.2, U2.2 (GND), U3.2 (GND), VCap1.2, VCap2.2, XL1.1 (P1), XL10.14 (GND), XL10.20 (GND), XL10.25 (GND), XL10.30 (GND), XL10.34 (GND), XL10.39 (GND), XL10.6 (GND), XL10.9 (GND), XL12.4 (UID), XL12.5 (UGND), XL2.3, XL3.1, XL5.2 (PM), XL6.2 (PM), XL9.A1 (GND), XL9.A12 (GND), XL9.B1 (GND), XL9.B12 (GND); no longer C1.1, C19.2, C44.2, C45.2, C46.2, C47.2, C48.2, C49.2, C50.2, C53.2, C54.2, C55.2, C57.2, R1.2, R48.2, U4.13 (PGND), U4.21 (DGND), U4.27 (PGND), U4.9 (AGND), U4.PAD, XL4.1 (P1)
- net MOTOR_CS: now also DA3.6 (Vo)
- net MOTOR_MISO: now also R30.2
- net MOTOR_MOSI: now also DA5.6 (Vo)
- net MOTOR_SCK: now also DA4.6 (Vo)
- net SWCLK: now also DD1.49 (SWCLK/(PA14)), XL2.2
- net SWDIO: now also DD1.46 (SWDIO/(PA13)), XL2.4
- net UART_RX: now also DD1.59 (PB7/SDA1/T4C2/RX1), XL2.6
- net UART_TX: now also DD1.58 (PB6/SCL1/T4C1/TX1), XL2.5
- net USB_D+: now also DD1.45 (OTGFS_DP/PA12); no longer R5.1
- net USB_D-: now also DD1.44 (OTGFS_DM/T1C4/PA11)
- net at XTAL1.1: now also C1.1, DD1.5 (PH0/OSCIN); no longer C10.1
- net at C18.2: now also DA1.6 (LX), L4.1
- net at R4.1: now also DD1.6 (PH1/OSCOUT)
- net at R4.2: now also XTAL1.2, C4.1
- net at R2.2: now also XL5.1 (P1); no longer C2.1
- net BUSY/SYNC_1 renamed BUSY/SYNC
- net BUSY/SYNC: now also R34.2
- net DIN+: no longer names the net of U1.3 (I/O2)
- net DIN+: now also L3.3; no longer XL7.3 (D+)
- net DIN-: no longer names the net of XL7.2 (D-)
- net DIN-: now also L3.1; no longer U1.1 (I/O1)
- net FLAG_1 renamed FLAG
- net FLAG: now also R33.2
- net STBY/RST renamed STBY/RST
- net STBY/RST: now also DA9.6 (Vo)
- net STEP_CLK_1 renamed STEP_CLK
- net SW_1 renamed SW
- net SW: now also DA8.6 (Vo); no longer R3.2
- net USB_PULLUP renamed +5v
- net +5v: now also C13.1, C14.1, C3.1, C6.1, D10.A, D13.A, D4.C, D9.A, DA1.5 (IN), Q4.1 (S), Q4.2 (S), Q4.3 (S), SW4.1, U2.5 (VBUS), XL1.2 (PM), XL9.A4 (VBUS), XL9.A9 (VBUS), XL9.B4 (VBUS), XL9.B9 (VBUS)
- net Vdd1 renamed VCC
- net VCC: now also C24.1, C28.1, C29.1, C30.1, C31.1, C32.1, C33.1, C34.1, DA2.7 (Ve), DA2.8 (Vcc), DA3.7 (Ve), DA3.8 (Vcc), DA4.7 (Ve), DA4.8 (Vcc), DA5.7 (Ve), DA5.8 (Vcc), DA6.7 (Ve), DA6.8 (Vcc), DA7.7 (Ve), DA7.8 (Vcc), DA8.7 (Ve), DA8.8 (Vcc), DA9.7 (Ve), DA9.8 (Vcc)
- new net: R12.1, XL8.2 (PM)
- new net: L3.2, U1.1 (I/O1)
- new net: L3.4, XL7.3 (D+)
- new net: C18.1, DA1.1 (BS)
- new net: C19.2, DA1.3 (FB), R10.1, R9.2
- new net: C17.1, DA1.4 (EN), R5.1
- new net: L1.1, XL7.H1
- new net: R1.2, XL4.1 (P1)
- new net: DD2.23 (R-EXT), R35.1
- new net: L6.1, XL9.S1 (PAD), XL9.S2 (PAD), XL9.S3 (PAD), XL9.S4 (PAD)
- new net: DD1.47 (VCap2), VCap2.1
- new net: DD1.42 ((OTGFS_VBUS)/T1C2/TX1/PA9), R15.1
- new net: D8.A, R6.2
- new net: DD1.61 (PB8/SDIO_D4/T4C3/T10C1/SCL1), R6.1
- new net: DD1.31 (VCap1), VCap1.1
- new net: R13.1, XL8.1 (P1)
- new net: U3.5 (VBUS), XL12.1 (UVcc)
- new net: L8.1, XL12.2 (D-)
- new net: L8.4, XL12.3 (D+)
- new net: L9.1, XL12.H1
- new net: L8.2, U3.1 (I/O1)
- new net: L8.3, U3.3 (I/O2)
- new net: Q1.3 (D), R8.2
- new net: D9.C, R8.1
- new net: R3.2, XL6.1 (P1)
- new net: D13.C, R18.1
- new net: Q3.3 (D), R18.2
- new net: D10.C, R14.1
- new net: Q2.3 (D), R14.2
- new net: DA3.2 (A), R20.1
- new net: L7.2, U2.1 (I/O1)
- new net: L7.3, U2.3 (I/O2)
- new net: DA4.2 (A), R21.1
- new net: DA5.2 (A), R22.1
- new net: DA2.2 (A), R30.1
- new net: DA7.2 (A), R34.1
- new net: DA8.2 (A), R31.1
- new net: DA6.2 (A), R33.1
- new net: DA9.2 (A), R32.1
- new net: C42.2, DD5.11 (VREG)
- new net: DD4.3 (2A), DD5.4 (CD)
- new net: C37.2, DD5.5 (~RSTN)
- new net: DD5.6 (EQ), R37.1
- new net: DD4.1 (1A), DD5.9 (ENA_HS)
- new net: DD4.4 (2Y), R41.1
- new net: DD4.6 (1Y), R40.1
- new net: D20.A, R40.2
- new net: D21.A, R41.2
- new net: D14.C, R19.1, SW1.1, SW2.1, SW3.1
- new net: R23.1, SW1.2
- new net: R24.1, SW2.2
- new net: R25.1, SW3.2
- new net: DD2.9 (Y4), VD1.1 (e)
- new net: DD2.8 (Y3), VD1.2 (d)
- new net: DD2.7 (Y2), VD1.3 (c)
- new net: DD2.6 (Y1), VD1.33 (b)
- new net: DD2.5 (Y0), VD1.34 (a)
- new net: DD2.11 (Y6), VD1.35 (g)
- new net: DD2.10 (Y5), VD1.36 (f)
- new net: DD2.12 (Y7), VD1.4 (DP)
- new net: DD2.14 (Y9), VD1.28 (b)
- new net: DD2.13 (Y8), VD1.29 (a)
- new net: DD2.18 (Y13), VD1.30 (f)
- new net: DD2.17 (Y12), VD1.5 (e)
- new net: DD2.16 (Y11), VD1.6 (d)
- new net: DD2.19 (Y14), VD1.7 (g)
- new net: DD2.15 (Y10), VD1.8 (c)
- new net: DD2.20 (Y15), VD1.9 (DP)
- new net: DD3.17 (Y12), VD1.14 (e)
- new net: DD3.16 (Y11), VD1.15 (d)
- new net: DD3.19 (Y14), VD1.16 (g)
- new net: DD3.15 (Y10), VD1.17 (c)
- new net: DD3.20 (Y15), VD1.18 (DP)
- new net: DD3.14 (Y9), VD1.19 (b)
- new net: DD3.13 (Y8), VD1.20 (a)
- new net: DD3.18 (Y13), VD1.21 (f)
- new net: DD3.9 (Y4), VD1.10 (e)
- new net: DD3.8 (Y3), VD1.11 (d)
- new net: DD3.7 (Y2), VD1.12 (c)
- new net: DD3.12 (Y7), VD1.13 (DP)
- new net: DD3.6 (Y1), VD1.24 (b)
- new net: DD3.5 (Y0), VD1.25 (a)
- new net: DD3.11 (Y6), VD1.26 (g)
- new net: DD3.10 (Y5), VD1.27 (f)
- new net: DD3.23 (R-EXT), R36.1
- new net: DD2.22 (DataOut), DD3.2 (DataIn)
- new net: Q4.4 (G), R26.1, SW4.2
- new net BUSY/SYNC_MCU: DA7.6 (Vo), DD1.11 ((ADC123-13)/MOSI2/PC3)
- new net Btn: C23.1, D11.C, R13.2, R17.1, XL10.36 (GPIO16)
- new net BtnDown: C26.1, D16.C, DD1.27 (PB1/T3C4/(ADC12-9)), R24.2, R28.1
- new net BtnFast: C27.1, D17.C, DD1.28 (PB2/BOOT1), R25.2, R29.1
- new net BtnUp: C25.1, D15.C, DD1.26 (PB0/T3C3/(ADC12-8)), R23.2, R27.1
- new net CLK: DD1.34 (PB13/SCK2), DD2.3 (CLK), DD3.3 (CLK)
- new net DATA_IN1: DD1.36 (PB15/MOSI2/T12C2), DD2.2 (DataIn)
- new net ENDSTOP_TOUCH: C11.1, D7.C, DD1.16 ((ADC123-2)/T5C3/T9C1/T2C3/TX2/PA2), R3.1
- new net FLAG_MCU: DA6.6 (Vo), DD1.25 ((ADC12-15)/PC5)
- new net GNDPWR: C28.2, C29.2, C30.2, C33.2, C34.2, C44.2, C45.2, C46.2, C47.2, C48.2, C49.2, C50.2, C53.2, C54.2, C55.2, C56.2, C57.2, C58.2, DA2.3 (C), DA3.5 (GND), DA4.5 (GND), DA5.5 (GND), DA6.3 (C), DA7.3 (C), DA8.5 (GND), DA9.5 (GND), HOLE1.H, HOLE2.H, R48.2, U4.13 (PGND), U4.21 (DGND), U4.27 (PGND), U4.9 (AGND), U4.PAD, XL13.1 (P1)
- new net Green: Q3.1 (G), R16.1, XL10.35 (GPIO19)
- new net LATCH: DD1.33 (PB12/CK3), DD2.4 (Latch), DD3.4 (Latch)
- new net MCU_RESET: DD1.7 (NRST), Q5.3 (D), R46.2
- new net MCU_RESET_CTRL: Q5.1 (G), R45.1, XL10.11 (GPIO17)
- new net MCU_RX_RPI_TX: DD1.52 (MISO3/RX4/RX3/SDIO_D3/PC11), XL10.8 (GPIO14/UART_TXD)
- new net MCU_TX_RPI_RX: DD1.51 (SCK3/TX4/TX3/SDIO_D2/PC10), XL10.10 (GPIO15/UART_RXD)
- new net MOTOR_CS_MCU: DD1.41 (MCO1/SCL3/T1C1/CK1/PA8), R20.2
- new net MOTOR_MISO_MCU: DA2.6 (Vo), DD1.22 ((ADC12-6)/T13C1/T3C1/MISO1/PA6)
- new net MOTOR_MOSI_MCU: DD1.23 ((ADC12-7)/T14C1/T3C2/MOSI1/PA7), R22.2
- new net MOTOR_SCK_MCU: DD1.21 ((ADC12-5)/(DAC2)/SCK1/PA5), R21.2
- new net OUT_EN: DD1.35 (PB14/MISO2/T12C1), DD2.21 (~OutEn), DD3.21 (~OutEn)
- new net PB3: DD1.57 (PB5/MOSI3/T3C2/MOSI1), XL3.2
- new net PB4: DD1.56 (PB4/MISO3/T3C1/MISO1), XL3.3
- new net PB5: DD1.55 (PB3/SCK3/T2C2/SCK1), XL3.4
- new net PWR_LEDS: C19.1, C20.1, C21.1, C22.1, C35.2, C36.2, C38.2, C39.2, DD2.24 (VCC), DD3.24 (VCC), L4.2, L5.2, R9.1, VD1.22 (CA), VD1.23 (CA), VD1.31 (CA), VD1.32 (CA)
- new net PWR_RPI: Q4.5 (D), Q4.6 (D), Q4.7 (D), Q4.8 (D), XL10.2 (5V), XL10.4 (5V)
- new net PwrMCU: C12.1, C15.1, C16.1, C2.1, C5.1, C7.1, C8.1, DD1.1 (VBAT), DD1.13 (VDDA), DD1.19 (VDD4), DD1.32 (VDD1), DD1.48 (VDD2), DD1.64 (VDD3), L2.1, XL2.1, XL3.5
- new net Red: Q1.1 (G), R7.1, XL10.40 (GPIO21)
- new net STBY/RST_MCU: DD1.10 ((ADC123-12)/MISO2/PC2), R32.2
- new net SW_MCU: DD1.24 ((ADC12-14)/PC4), R31.2
- new net USB2_C_DM: L7.1, XL9.A7 (D-), XL9.B7 (D-)
- new net USB2_C_DP: L7.4, XL9.A6 (D+), XL9.B6 (D+)
- new net USB2_D+: DD5.2 (D1P), DD5.7 (D2P), U2.4 (I/O2), U3.4 (I/O2)
- new net USB2_D-: DD5.1 (D1M), DD5.8 (D2M), U2.6 (I/O1), U3.6 (I/O1)
- new net Yellow: Q2.1 (G), R11.1, XL10.38 (GPIO20)
- no-connect marks 37 -> 22
Other:
- note added: "+12v"
- note added: "+5v and +3v3"
- note added: "Endstops"
- note added: "External +5V or USB"
- note added: "LED Display"
- note added: "MCU Reset"
- note added: "Motor Control Buttons"
- note added: "Motor Driver"
- note added: "Optocouplers"
- note added: "Raspberry"
- note added: "Raspberry PWR Reset"
- note added: "Red Green Yellow Indication"
- note added: "Start Button"
- note added: "USB for MCU"
- note added: "USB-C for Mini"
- note added: "uUSB for Raspberry to Mini"
- note removed: "USB connector with protection\n"
- moved on the sheet: C3, C44, C45, C46, C47, C48, C49, C50, C51, C52, C53, C54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

Commit message: PCB sent to factory
Parts:
- removed TP4: TESTPOINT, PCB:TESTPOINT_1MM, symbol pcb_details:TESTPOINT
- added C33: 0.1u, Capacitors:CAP_0603_Silks, symbol Tittar_kl:C
- added D18, D19: PESD3V3, Diodes:SOD323, symbol Tittar_kl:ZenerBidir
- added R31, R32: 1k, Resistors:RES_0603, symbol Tittar_kl:R
- added R35: 100k, Resistors:RES_0603, symbol Tittar_kl:R
- added XL10: CONN_2, Connectors:WB-02(MW-2M), symbol Connectors_kl:CONN_2
- added XL15: CONN_1, Connectors:PLS-1Rnd, symbol Connectors_kl:CONN_1
- C13, C20, C21: footprint Capacitors:CAP_0603 -> Capacitors:CAP_0805
- C14, C17, C18, C19, C22: footprint Capacitors:CAP_0402 -> Capacitors:CAP_0603_Silks
- C23, C25, C26, C27, C3, VCap1, VCap2: footprint Capacitors:CAP_0603 -> Capacitors:CAP_0603_Silks
- C36: renamed from C35; footprint Capacitors:CAP_0402 -> Capacitors:CAP_0603_Silks
- C37: renamed from C36; footprint Capacitors:CAP_0402 -> Capacitors:CAP_0603_Silks
- C38: renamed from C37; footprint Capacitors:CAP_0603 -> Capacitors:CAP_0603_Silks
- C39: renamed from C38; footprint Capacitors:CAP_0603 -> Capacitors:CAP_0805
- C40: renamed from C39; footprint Capacitors:CAP_0603 -> Capacitors:CAP_0805
- C41: renamed from C40; footprint Capacitors:CAP_0603 -> Capacitors:CAP_0603_Silks
- C42: renamed from C41; footprint Capacitors:CAP_0603 -> Capacitors:CAP_0603_Silks
- C43: renamed from C42; footprint Capacitors:CAP_0603 -> Capacitors:CAP_0603_Silks
- C44: renamed from C43; footprint Capacitors:CAP_0603 -> Capacitors:CAP_0603_Silks
- C45: renamed from C44; footprint Capacitors:CAP_0603 -> Capacitors:CAP_0603_Silks
- C46: renamed from C45; footprint Capacitors:CAP_0603 -> Capacitors:CAP_0603_Silks
- C47: renamed from C46; footprint Capacitors:CAP_0603 -> Capacitors:CAP_0603_Silks
- C48: renamed from C47; footprint Capacitors:CAP_0603 -> Capacitors:CAP_0603_Silks
- C49: renamed from C48; footprint Capacitors:CAP_0603 -> Capacitors:CAP_0603_Silks
- C52: renamed from C51; footprint Capacitors:CAP_0603 -> Capacitors:CAP_0603_Silks
- C53: renamed from C52; footprint Capacitors:CAP_0603 -> Capacitors:CAP_0603_Silks
- C54: renamed from C53; footprint Capacitors:CAP_0603 -> Capacitors:CAP_0603_Silks
- C55: renamed from C54; footprint Capacitors:CAP_0603 -> Capacitors:CAP_0603_Silks
- C56: renamed from C55; footprint Capacitors:CAP_0603 -> Capacitors:CAP_0603_Silks
- C58: renamed from C57; footprint Capacitors:CAP_0603 -> Capacitors:CAP_0603_Silks
- C59: renamed from C58; footprint Capacitors:CAP_0603 -> Capacitors:CAP_0603_Silks
- DA2, DA3, DA4, DA5, DA6, DA7, DA8, DA9: footprint (none) -> DIP:DIP-8_296_ELL
- DD1: footprint (none) -> LQFP_TQFP:LQFP64
- DD4: footprint (none) -> SOT:SOT23-6
- Q1, Q2, Q3, Q5: footprint (none) -> SOT:SOT23-3
- R10, R5, R9: footprint Resistors:RES_0402_sm -> Resistors:RES_0603
- R38: renamed from R35; footprint Resistors:RES_0402_sm -> Resistors:RES_0603
- R39: renamed from R36; footprint Resistors:RES_0402_sm -> Resistors:RES_0603
- XL1: footprint (none) -> Connectors:2ZHDRC-02P
- XL13: renamed from XL12; symbol Connectors_kl:USB_MICRO_2H -> Connectors_kl:USB_MICRO_4H
- XL14: renamed from XL13; footprint (none) -> Connectors:2ZHDRC-02P
- XL7: symbol Connectors_kl:USB_MICRO_2H -> Connectors_kl:USB_MICRO_4H
- XL9: footprint (none) -> Connectors:USB_C_MOLEX_1054500101; PN (none) -> Molex 1054500101
- renumbered C33 to C34, C34 to C35, C49 to C50, C50 to C51, C56 to C57, D18 to D20, D19 to D21, D20 to D22, D21 to D23, D22 to D24, D23 to D25, R31 to R33, R32 to R34, R33 to R36, R34 to R37, R37 to R40, R38 to R41, R39 to R42, R40 to R43, R41 to R44, R42 to R45, R43 to R46, R44 to R47, R45 to R48, R46 to R49, R47 to R50, R48 to R51, XL10 to XL11, XL11 to XL12
Connections:
- net +3v3: now also C24.1, C31.1, C32.1, DA2.7 (Ve), DA2.8 (Vcc), DA6.7 (Ve), DA6.8 (Vcc), DA7.7 (Ve), DA7.8 (Vcc), D19.C, R31.2; no longer R49.1
- net GND: now also XL11.H (Housing), C33.2, D18.A, D19.A, R35.2, XL15.1 (P1); no longer HOLE3.H, HOLE4.H, HOLE5.H, HOLE6.H
- net PwrMCU: now also R49.1
- net USB2_C_DM: now also L7.4; no longer L7.1
- net USB2_C_DP: now also L7.1; no longer L7.4
- net USB2_D+: now also U2.6 (I/O1); no longer U2.4 (I/O2)
- net USB2_D-: now also U2.4 (I/O2); no longer U2.6 (I/O1)
- net VCC: no longer C24.1, C31.1, C32.1, DA2.7 (Ve), DA2.8 (Vcc), DA6.7 (Ve), DA6.8 (Vcc), DA7.7 (Ve), DA7.8 (Vcc)
- net at L1.1, XL7.H1: now also XL7.H2, XL7.H3, XL7.H4
- net at L9.1, XL13.H1: now also XL13.H2, XL13.H3, XL13.H4
- net ChClosed: now reaches DD1.29 (PB10/SCK2/SCL2/TX3/T2C3)
- net ChClosed: now also C33.1, D18.C, R32.2, R35.1
- net STEP_CLK: no longer names the net of U4.25 (STCK)
- new net: R31.1, XL10.2 (PM)
- new net: R32.1, XL10.1 (P1)
- no-connect marks 22 -> 62
Other:
- note added: "Chamber Closed Button"
- moved on the sheet: TP1, TP2, TP3

Commit message: Proceeding with business logic
Parts:
- removed R36, R37: 1k, Resistors:RES_0603, symbol Tittar_kl:R
- added C? (x5): 0.1u, Capacitors:CAP_0603_Silks, symbol Tittar_kl:C
- added C? (x2): 18pF, Capacitors:CAP_0603_Silks, symbol Tittar_kl:C
- added C?: 10u, Capacitors:CAP_0805, symbol Tittar_kl:C
- added C?: 1u, Capacitors:CAP_0603_Silks, symbol Tittar_kl:C
- added D?: LED, LEDs:LED_0603, symbol Tittar_kl:LED
- added DD?: STM32L476Rx, LQFP_TQFP:LQFP64, symbol st_kl:STM32L476Rx
- added L?: BLM15AG102, Inductors:IND_0402, symbol Tittar_kl:L
- added R? (x3): 1k, Resistors:RES_0603, symbol Tittar_kl:R
- added R? (x4): 4k7, Resistors:RES_0603, symbol Tittar_kl:R
- added XTAL?: 12 MHz, Quartz:03225C4, symbol Tittar_kl:CRYSTAL_H
- R45, R46: value 56k -> 1k
Connections:
- net +3v3: now also L?.2
- net 5V_USB: now also R?.2
- net BUSY/SYNC: now also DA7.2 (A)
- net BUSY/SYNC_MCU: now also DD?.11 (ADC123-4/MOSI2/PC3)
- net BtnDown: now also DD?.27 (PB1/T3C4/QSPI0/LPTIM2_IN1/ADC12-16)
- net BtnFast: now also DD?.28 (PB2/LPTIM1_OUT/RTC_OUT)
- net BtnUp: now also DD?.26 (PB0/T3C3/QSPI1/ADC12-15)
- net CLK: now also DD?.34 (PB13/SCK2/SCL2)
- net ChClosed: now also DD?.29 (PB10/T2C3/SCK2/SCL2/TX3/LPRX1/QSPI_CLK)
- net DATA_IN1: now also DD?.36 (PB15/MOSI2/T15C2)
- net ENDSTOP_BOT: now also DD?.14 (ADC12-5/WKUP1/T2C1/T5C1/TX4/PA0)
- net ENDSTOP_TOP: now also DD?.15 (ADC12-6/T2C2/T5C2/RX4/PA1)
- net ENDSTOP_TOUCH: now also DD?.16 (ADC12-7/WKUP4/T15C1/T2C3/T5C3/TX2/PA2)
- net FLAG: now also DA6.2 (A)
- net FLAG_MCU: now also DD?.25 (ADC12-14/RX3/PC5)
- net GND: now also C?.2, C?.2, C?.2, C?.2, C?.2, C?.2, C?.2, C?.2, C?.2, DD?.12 (VSSA/VREF-), DD?.18 (VSS), DD?.31 (VSS), DD?.47 (VSS), DD?.60 (BOOT0), DD?.63 (VSS), XTAL?.H
- net LATCH: now also DD?.33 (PB12/CK3)
- net MCU_RESET: now also DD?.7 (NRST)
- net MCU_RX_RPI_TX: now also DD?.52 (MISO3/RX4/RX3/SDIO_D3/PC11)
- net MCU_TX_RPI_RX: now also DD?.51 (SCK3/TX4/TX3/SDIO_D2/PC10)
- net MOTOR_CS: now also R?.2
- net MOTOR_CS_MCU: now also DD?.41 (OTG_SOF/LPTIM2_OUT/MCO/T1C1/CK1/PA8)
- net MOTOR_MISO_MCU: now also DD?.22 (ADC12-11/T3C1/T16C1/QSPI3/MISO1/PA6)
- net MOTOR_MOSI: now also R?.2
- net MOTOR_MOSI_MCU: now also DD?.23 (ADC12-12/T3C2/T17C1/QSPI2/MOSI1/PA7)
- net MOTOR_SCK: now also R?.2
- net MOTOR_SCK_MCU: now also DD?.21 (ADC12-10/T2C1/DAC2/SCK1/PA5)
- net OUT_EN: now also DD?.35 (PB14/MISO2/SDA2/T15C1)
- net PB3: now also DD?.57 (PB5/MOSI1/MOSI3/T3C2/CK1/LPTIM1_IN1)
- net PB4: now also DD?.56 (PB4/MISO1/MISO3/T3C1)
- net PB5: now also DD?.55 (PB3/SCK1/SCK3/T2C2/SWO)
- net PwrMCU: now also C?.1, C?.1, C?.1, C?.1, C?.1, C?.1, C?.1, DD?.1 (VBAT), DD?.13 (VDDA/VREF+), DD?.19 (VDD), DD?.32 (VDD), DD?.48 (VDDUSB), DD?.64 (VDD), L?.1
- net STBY/RST: now also R?.2
- net STBY/RST_MCU: now also DD?.10 (ADC123-3/LPTIM1_IN2/MISO2/PC2)
- net SWCLK: now also DD?.49 (SWCLK/PA14)
- net SWDIO: now also DD?.46 (SWDIO/PA13)
- net SW_MCU: now also DD?.24 (ADC12-13/TX3/PC4)
- net UART_RX: now also DD?.59 (PB7/SDA1/T4C2/RX1/LPTIM1_IN2)
- net UART_TX: now also DD?.58 (PB6/SCL1/T4C1/TX1)
- net USB_D+: now also DD?.45 (OTG_DP/PA12)
- net USB_D-: now also DD?.44 (OTG_DM/T1C4/PA11)
- net VCC: now also R?.1, R?.1, R?.1, R?.1
- new net: C?.1, DD?.5 (PH0/OSCIN), XTAL?.1
- new net: C?.1, R?.2, XTAL?.2
- new net: DD?.42 (OTG_VBUS/T1C2/TX1/PA9), R?.1
- new net: DD?.61 (PB8/SDIO_D4/T4C3/T16C1/SCL1), R?.1
- new net: D?.A, R?.2
- new net: DD?.6 (PH1/OSCOUT), R?.1
- no-connect marks 62 -> 79
Other:
- moved on the sheet: C24, C28, C29, C30, C31, C32, C34, DA2, DA3, DA4, DA5, DA6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
